Commit message: adjust config

File: src/amiga_sim/urdf/amiga_model_v1.urdf (robot description, URDF)
Before this commit: robot amiga_model, 24 links, 23 joints
Links:
- removed link camera_mount_plate_link
- removed link camera_mount_tube_link
- removed link lower_mount_plate_link
- removed link oak_d_camera_1_link
- removed link oak_d_camera_2_link
- added link extra_tube_plate_e_link, mass 0; collision mesh filename=package://amiga_sim/meshes/extra_tube_plate_link.STL; visual mesh filename=package://amiga_sim/meshes/extra_tube_plate_link.STL
- added link extra_tube_plate_f_link, mass 0; collision mesh filename=package://amiga_sim/meshes/extra_tube_plate_link.STL; visual mesh filename=package://amiga_sim/meshes/extra_tube_plate_link.STL
- added link oak_d_camera_1_tube_plate_link, mass 0; collision mesh filename=package://amiga_sim/meshes/extra_tube_plate_link.STL; visual mesh filename=package://amiga_sim/meshes/extra_tube_plate_link.STL
Joints:
- removed joint camera_mount_plate_joint
- removed joint camera_mount_tube_joint
- removed joint lower_mount_plate_joint
- removed joint oak_d_camera_1_joint
- removed joint oak_d_camera_2_joint
- added joint extra_tube_plate_e_joint: type fixed, parent base_link, child extra_tube_plate_e_link, origin xyz=0.602415 1.31441 0.78102 rpy=1.5708 -1.5708 1.5708, axis 0 0 0
- added joint extra_tube_plate_f_joint: type fixed, parent base_link, child extra_tube_plate_f_link, origin xyz=0.602415 1.32741 0.78102 rpy=0 0 0, axis 0 0 0
- added joint oak_d_camera_1_tube_plate_joint: type fixed, parent intelligence_kit_link, child oak_d_camera_1_tube_plate_link, origin xyz=-0.01 -0.2 0 rpy=1.5708 1.5708 0, axis 0 0 0
- joint brain_joint: origin xyz=0.0438125 -0.0134064575902699 -0.13786349367425 rpy=2.44346095279172 0 3.14159265358979 -> xyz=0.0438125 0.4004575902699 -0.13786349367425 rpy=2.44346095279172 0 3.14159265358979
- joint intelligence_kit_joint: origin xyz=0.47409121329226 -0.36658102124713 1.02035935922013 rpy=1.5707963267949 0 3.14159265358979 -> xyz=0.602415 1.34041 1.1702 rpy=1.5707963267949 0 3.14159265358979
- joint poe_switch_joint: origin xyz=0.01016 0.15460290397814 0 rpy=1.5707963267949 -1.5707963267949 0 -> xyz=0.01016 0.22060290397814 0 rpy=-1.5708 0 0

Commit message: adjust config

File: src/amiga_sim/urdf/amiga_model_v1.urdf (robot description, URDF)
Before this commit: robot amiga_model, 22 links, 21 joints
Joints:
- joint dash_mast_joint: origin xyz=1.002 1.18340602124668 1.0010200092266 rpy=0.523598692765961 -0.000309268842448867 -3.1416 -> xyz=0.942 1.18340602124668 1.0010200092266 rpy=0.523598692765961 -0.000309268842448867 -3.1416

Commit message: implement camera 2

File: src/amiga_sim/urdf/amiga_model_v1.urdf (robot description, URDF)
Before this commit: robot amiga_model, 22 links, 21 joints
Links:
- removed link oak_d_camera_1_tube_plate_link
- added link oak_d_camera_2_link, mass 0.0415063479146466; collision mesh filename=package://amiga_sim/meshes/oak_d_camera_2_link.STL; visual mesh filename=package://amiga_sim/meshes/oak_d_camera_2_link.STL
- added link oak_d_camera_2_mount_link, mass 0.026503699588838; collision mesh filename=package://amiga_sim/meshes/lower_mount_plate_link.STL scale=1.4 1 1; visual mesh filename=package://amiga_sim/meshes/lower_mount_plate_link.STL scale=1.4 1 1
- added link oak_d_camera_2_tube_plate_link, mass 0; collision mesh filename=package://amiga_sim/meshes/extra_tube_plate_link.STL; visual mesh filename=package://amiga_sim/meshes/extra_tube_plate_link.STL
Joints:
- removed joint oak_d_camera_1_tube_plate_joint
- added joint oak_d_camera_2_joint: type fixed, parent oak_d_camera_2_mount_link, child oak_d_camera_2_link, origin xyz=-0.05 0.022 0.01 rpy=0 0 0, axis 0 0 0
- added joint oak_d_camera_2_mount_joint: type fixed, parent oak_d_camera_2_tube_plate_link, child oak_d_camera_2_mount_link, origin xyz=-0.05 -0.073 0 rpy=-1.5708 0 1.5708, axis 0 0 0
- added joint oak_d_camera_2_tube_plate_joint: type fixed, parent intelligence_kit_link, child oak_d_camera_2_tube_plate_link, origin xyz=-0.01 -0.2 0 rpy=1.5708 1.5708 0, axis 0 0 0

Commit message: horizontal mount

File: src/amiga_sim/urdf/amiga_model_v1.urdf (robot description, URDF)
Before this commit: robot amiga_model, 24 links, 23 joints
Links:
- added link horizontal_module_tube_link, mass 0.416973913768598; collision mesh filename=package://amiga_sim/meshes/long_extra_tube_link.STL scale=1 0.85 1; visual mesh filename=package://amiga_sim/meshes/long_extra_tube_link.STL scale=1 0.85 1
- added link horizontal_module_tube_plate_a_link, mass 0; collision mesh filename=package://amiga_sim/meshes/extra_tube_plate_link.STL; visual mesh filename=package://amiga_sim/meshes/extra_tube_plate_link.STL
- added link horizontal_module_tube_plate_b_link, mass 0; collision mesh filename=package://amiga_sim/meshes/extra_tube_plate_link.STL; visual mesh filename=package://amiga_sim/meshes/extra_tube_plate_link.STL
- link long_extra_tube_link: mass 0.151244220009192 -> 0.416973913768598
Joints:
- added joint horizontal_module_tube_joint: type fixed, parent horizontal_module_tube_plate_b_link, child horizontal_module_tube_link, origin xyz=0 0.012 0.07 rpy=1.5708 0 0, axis 0 0 0
- added joint horizontal_module_tube_plate_a_joint: type fixed, parent intelligence_kit_link, child horizontal_module_tube_plate_a_link, origin xyz=0.01 -0.07 0 rpy=-1.5708 1.5708 0, axis 0 0 0
- added joint horizontal_module_tube_plate_b_joint: type fixed, parent horizontal_module_tube_plate_a_link, child horizontal_module_tube_plate_b_link, origin xyz=0 -0.014 0 rpy=3.1416 1.5708 0, axis 0 0 0

Commit message: adjustment

File: src/amiga_sim/urdf/amiga_model_v1.urdf (robot description, URDF)
Before this commit: robot amiga_model, 27 links, 26 joints
Links:
- link intelligence_kit_link: geometry collision mesh filename=package://amiga_sim/meshes/intelligence_kit_link.STL scale=1 0.91 1; visual mesh filename=package://amiga_sim/meshes/intelligence_kit_link.STL scale=1 0.91 1
Joints:
- joint brain_joint: origin xyz=0.0438125 0.4004575902699 -0.13786349367425 rpy=2.44346095279172 0 3.14159265358979 -> xyz=0.0438125 0.3404575902699 -0.13786349367425 rpy=2.44346095279172 0 3.14159265358979
- joint poe_switch_joint: origin xyz=0.01016 0.22060290397814 0 rpy=-1.5708 0 0 -> xyz=0.01016 0.17060290397814 0 rpy=-1.5708 0 0

Commit message: adjust config

File: src/amiga_sim/urdf/amiga_model_v1.urdf (robot description, URDF)
Before this commit: robot amiga_model, 27 links, 26 joints
Links:
- link intelligence_kit_link: geometry collision mesh filename=package://amiga_sim/meshes/intelligence_kit_link.STL scale=1 0.87 1; visual mesh filename=package://amiga_sim/meshes/intelligence_kit_link.STL scale=1 0.87 1
Joints:
- joint horizontal_module_tube_plate_a_joint: origin xyz=0.01 -0.07 0 rpy=-1.5708 1.5708 0 -> xyz=0.01 -0.078 0 rpy=-1.5708 1.5708 0
- joint intelligence_kit_joint: origin xyz=0.602415 1.34041 1.1702 rpy=1.5707963267949 0 3.14159265358979 -> xyz=0.602415 1.34041 1.1402 rpy=1.5707963267949 0 3.14159265358979

Commit message: adjust config

File: src/amiga_sim/urdf/amiga_model_v1.urdf (robot description, URDF)
Before this commit: robot amiga_model, 27 links, 26 joints
Joints:
- joint brain_joint: origin xyz=0.0438125 0.3404575902699 -0.13786349367425 rpy=2.44346095279172 0 3.14159265358979 -> xyz=0.0438125 0.3354575902699 -0.13786349367425 rpy=2.44346095279172 0 3.14159265358979

Commit message: adjust config

File: src/amiga_sim/urdf/amiga_model_v1.urdf (robot description, URDF)
Before this commit: robot amiga_model, 27 links, 26 joints
Links:
- added link oak_d_camera_1_sub_mount_link, mass 0.026503699588838; collision mesh filename=package://amiga_sim/meshes/lower_mount_plate_link.STL scale=1.4 1 1; visual mesh filename=package://amiga_sim/meshes/lower_mount_plate_link.STL scale=1.4 1 1
- added link oak_d_camera_1_tube_plate_link, mass 0; collision mesh filename=package://amiga_sim/meshes/extra_tube_plate_link.STL; visual mesh filename=package://amiga_sim/meshes/extra_tube_plate_link.STL
Joints:
- added joint oak_d_camera_1_sub_mount_joint: type fixed, parent oak_d_camera_1_tube_plate_link, child oak_d_camera_1_sub_mount_link, origin xyz=0 -0.01 0 rpy=1.5708 -1.5708 0, axis 0 0 0
- added joint oak_d_camera_1_tube_plate_joint: type fixed, parent horizontal_module_tube_link, child oak_d_camera_1_tube_plate_link, origin xyz=0 0.35 -0.01 rpy=1.5708 0 0, axis 0 0 0

Commit message: adjust config

File: src/amiga_sim/urdf/amiga_model_v1.urdf (robot description, URDF)
Before this commit: robot amiga_model, 29 links, 28 joints
Links:
- removed link oak_d_camera_1_sub_mount_link
- added link oak_d_camera_1_base_mount_link, mass 0.026503699588838; collision mesh filename=package://amiga_sim/meshes/lower_mount_plate_link.STL scale=1.12 1 1; visual mesh filename=package://amiga_sim/meshes/lower_mount_plate_link.STL scale=1.12 1 1
- added link oak_d_camera_1_mount_link, mass 0.026503699588838; collision mesh filename=package://amiga_sim/meshes/lower_mount_plate_link.STL scale=1.4 1 1; visual mesh filename=package://amiga_sim/meshes/lower_mount_plate_link.STL scale=1.4 1 1
Joints:
- removed joint oak_d_camera_1_sub_mount_joint
- added joint oak_d_camera_1_base_mount_joint: type fixed, parent oak_d_camera_1_tube_plate_link, child oak_d_camera_1_base_mount_link, origin xyz=0 -0.01 0 rpy=1.5708 -1.5708 0, axis 0 0 0
- added joint oak_d_camera_1_mount_joint: type fixed, parent oak_d_camera_1_base_mount_link, child oak_d_camera_1_mount_link, origin xyz=0 -0.023 0.06 rpy=-1.5708 1.5708 0, axis 0 0 0

Commit message: full assembly

File: src/amiga_sim/urdf/amiga_model_v1.urdf (robot description, URDF)
Before this commit: robot amiga_model, 30 links, 29 joints
Links:
- added link oak_d_camera_1_link, mass 0.0415063479146466; collision mesh filename=package://amiga_sim/meshes/oak_d_camera_1_link.STL; visual mesh filename=package://amiga_sim/meshes/oak_d_camera_1_link.STL
Joints:
- added joint oak_d_camera_1_joint: type fixed, parent oak_d_camera_1_mount_link, child oak_d_camera_1_link, origin xyz=0.055 -0.045 -0.02 rpy=3.1416 0 1.5708, axis 0 0 0

Commit message: adjust config

File: src/amiga_sim/urdf/amiga_model_v1.urdf (robot description, URDF)
Before this commit: robot amiga_model, 31 links, 30 joints
Joints:
- joint dash_mast_joint: origin xyz=0.942 1.18340602124668 1.0010200092266 rpy=0.523598692765961 -0.000309268842448867 -3.1416 -> xyz=0.878 1.18340602124668 1.0010200092266 rpy=0.523598692765961 -0.000309268842448867 -3.1416
- joint oak_d_camera_1_joint: origin xyz=0.055 -0.045 -0.02 rpy=3.1416 0 1.5708 -> xyz=0.05 -0.045 -0.02 rpy=3.1416 0 1.5708

Commit message: add logo

File: src/amiga_sim/urdf/amiga_model_v1.urdf (robot description, URDF)
Before this commit: robot amiga_model, 31 links, 30 joints
Links:
- added link i_logo_link, mass 0; collision mesh filename=package://amiga_sim/meshes/i_logo_link.STL scale=0.4 0.4 0.4; visual mesh filename=package://amiga_sim/meshes/i_logo_link.STL scale=0.4 0.4 0.4
- added link i_logo_outer_link, mass 0; collision mesh filename=package://amiga_sim/meshes/i_logo_outer_link.STL scale=0.4 0.4 0.4; visual mesh filename=package://amiga_sim/meshes/i_logo_outer_link.STL scale=0.4 0.4 0.4
Joints:
- added joint i_logo_joint: type fixed, parent base_link, child i_logo_link, origin xyz=1.043 0.95447 0.62506 rpy=0 0 1.5708, axis 0 0 0
- added joint i_logo_outer_joint: type fixed, parent base_link, child i_logo_outer_link, origin xyz=1.043 0.95447 0.62506 rpy=0 0 1.5708, axis 0 0 0

Commit message: adjust joint pos

File: src/amiga_sim/urdf/amiga_model_v1.urdf (robot description, URDF)
Before this commit: robot amiga_model, 33 links, 32 joints
Joints:
- joint bl_wheel_joint: origin xyz=0.27384 -0.15588 0.42506 rpy=-1.5708 0 -1.5708 -> xyz=0.27384 -0.15588 0.42916 rpy=-1.5708 0 -1.5708
- joint br_wheel_joint: origin xyz=0.91244 -0.14953 0.42506 rpy=1.5708 0 1.5708 -> xyz=0.91244 -0.14953 0.42916 rpy=1.5708 0 1.5708
- joint fl_wheel_joint: origin xyz=0.27384 0.94812 0.42506 rpy=-1.5708 0 -1.5708 -> xyz=0.27384 0.94812 0.42916 rpy=-1.5708 0 -1.5708
- joint fr_wheel_joint: origin xyz=0.91244 0.95447 0.42506 rpy=1.5708 0 1.5708 -> xyz=0.91244 0.95447 0.42916 rpy=1.5708 0 1.5708

Commit message: physics adjustment

File: src/amiga_sim/urdf/amiga_model_v1.urdf (robot description, URDF)
Before this commit: robot amiga_model, 33 links, 32 joints
Links:
- link base_link: mass 86.4440274940804 -> 16.4440274940804

Commit message: add base footprint link

File: src/amiga_sim/urdf/amiga_model_v1.urdf (robot description, URDF)
Before this commit: robot amiga_model, 33 links, 32 joints
Links:
- added link base_footprint, mass 16.4440274940804; collision mesh filename=package://amiga_sim/meshes/base_link.STL; visual mesh filename=package://amiga_sim/meshes/base_link.STL
- link base_link: mass 16.4440274940804 -> None; geometry 
Joints:
- added joint base_joint: type fixed, parent base_link, child base_footprint, origin xyz=-0.6 -0.5 0 rpy=0 0 0
- joint bl_wheel_joint: parent base_link -> base_footprint
- joint br_wheel_joint: parent base_link -> base_footprint
- joint dash_mast_joint: parent base_link -> base_footprint
- joint extra_tube_a_joint: parent base_link -> base_footprint
- joint extra_tube_b_joint: parent base_link -> base_footprint
- joint extra_tube_c_joint: parent base_link -> base_footprint
- joint extra_tube_d_joint: parent base_link -> base_footprint
- joint extra_tube_plate_a_joint: parent base_link -> base_footprint
- joint extra_tube_plate_b_joint: parent base_link -> base_footprint
- joint extra_tube_plate_c_joint: parent base_link -> base_footprint
- joint extra_tube_plate_d_joint: parent base_link -> base_footprint
- joint extra_tube_plate_e_joint: parent base_link -> base_footprint
- joint extra_tube_plate_f_joint: parent base_link -> base_footprint
- joint fl_wheel_joint: parent base_link -> base_footprint
- joint fr_wheel_joint: parent base_link -> base_footprint
- joint i_logo_joint: parent base_link -> base_footprint
- joint i_logo_outer_joint: parent base_link -> base_footprint
- joint intelligence_kit_joint: parent base_link -> base_footprint
- joint long_extra_tube_joint: parent base_link -> base_footprint
- joint oak_d_camera_3_joint: parent base_link -> base_footprint
